Commit message: PR06: fix to base_link

File: src/course_description/urdf/vehicle.urdf.xacro (robot description, xacro)
@@ -53,5 +53,5 @@
   </link>
   <joint name="lidar_joint" type="fixed">
-    <parent link="camera_link"/>
+    <parent link="base_link"/>
     <child  link="lidar_link"/>
     <origin xyz="${lidar_xyz}" rpy="0 0 0"/>
